Commit message: Update controllers and xacro environment

File: urdf/robotiq_gripper.xacro (robot description, xacro)
@@ -35,5 +35,5 @@
           <color rgba="0.1 0.1 0.1 1" />
         </material>
-      </visual>
+      </visual>tool0_eoa
       <collision>
         <geometry>

File: urdf/workcell.urdf.xacro (robot description, xacro)
@@ -3,5 +3,5 @@
   <xacro:property name="ur_prefix" value="" />
   <!-- Xacro for the table -->
-  <xacro:include filename="$(find conntact)/urdf/assembly_table.xacro"/>
+  <!-- <xacro:include filename="$(find conntact)/urdf/assembly_table.xacro"/> -->
   <!-- Xacros from the Siemens Gear Assembly Challenge -->
 <!--  <xacro:include filename="$(find assembly_ros)/support/urdf/siemens_base_plate.xacro"/>
@@ -9,5 +9,5 @@
   <xacro:include filename="$(find assembly_ros)/support/urdf/siemens_big_shaft.xacro"/>-->
 <!-- Xacros from the NIST Task Board #1-->
-  <xacro:include filename="$(find conntact)/urdf/laser_cut_base_plate.xacro"/>
+  <!-- <xacro:include filename="$(find conntact)/urdf/laser_cut_base_plate.xacro"/> -->
   <!-- OLD FROM AUTOASSEMBLY Xacro for UR10e -->
 <!--  <xacro:include filename="$(find ur_e_description)/urdf/ur10e.urdf.xacro"/>-->
@@ -15,11 +15,11 @@
   <xacro:include filename="$(find ur_description)/urdf/ur10e.xacro"/>
   <!-- Xacro for gripper -->
-  <xacro:include filename="$(find conntact)/urdf/robotiq_gripper.xacro"/>
+  <!-- <xacro:include filename="$(find conntact)/urdf/robotiq_gripper.xacro"/> -->
 <!--  TODo: My Addition-->
-  <xacro:robotiq_gripper parent="tool0"/>
+  <!-- <xacro:robotiq_gripper parent="tool0"/> -->
   <!-- Static environment -->
 <!--  <link name="world"/>-->
 <!--  <xacro:assembly_table parent="world"/>-->
-  <xacro:assembly_table parent="base_link"/>
+  <!-- <xacro:assembly_table parent="base_link"/> -->
 <!--  <xacro:laser_cut_base_plate parent="table">
     <origin xyz="0.4 -0.7 0.0" rpy="-0.0091 -0.013 0.0197"/>
